Commit message: Delete extra files

File: panthera_python/Panthera-HT_description/urdf/Panthera-HT_description_follower.urdf (robot description, URDF)
Before this commit: robot Panthera-HT_description, 8 links, 7 joints
Links:
- link link6: mass 0.30 -> 0.32

File: panthera_python/Panthera-HT_description/urdf/Panthera-HT_description_with_finger.urdf (robot description, URDF)
Before this commit: robot Panthera-HT_description, 9 links, 8 joints
Links:
- link link6: mass 0.45 -> 0.32
